File: boards/simpleadapter/simpleadapter.kicad_pcb (KiCad board)
At the start: 2 copper layers, 14.2 x 17.3 mm, 2 parts, among them J1 692112030100-fixed, J2 Conn_02x05_Odd_Even

Commit message: New
Parts:
- J2: footprint Connector_PinSocket_2.54mm:PinSocket_2x05_P2.54mm_Vertical -> Connector_PinHeader_2.54mm:PinHeader_2x05_P2.54mm_Vertical
- moved J2 2.43 mm to (158.4, 99.6)
Routing:
- net /DRAIN: track 4.33 -> 7.82 mm
- net /SSTX+: track 4.78 -> 8.25 mm
- net /SSTX-: track 4.55 -> 8.02 mm
- net /GND: track 7.76 -> 4.50 mm
- net /SSRX+: track 4.55 -> 7.58 mm
- net /VBUS: track 7.76 -> 5.17 mm
- net /SSRX-: track 4.88 -> 7.35 mm
- net /D+: track 7.41 -> 4.93 mm
- net /D-: track 7.51 -> 5.16 mm
- net /SHIELD: track 24.2 -> 22.4 mm
Other:
- board text added: "1"
