File: boards/simpleadapter/simpleadapter.kicad_sch (KiCad schematic)
At the start: 2 parts, among them J1 692112030100, J2 Conn_02x05_Odd_Even

Commit message: Move to 14 pin headers for switch with off-board adapters
Parts:
- J2: footprint Connector_PinSocket_2.54mm:PinSocket_2x05_P2.54mm_Vertical -> Connector_PinHeader_2.54mm:PinHeader_2x05_P2.54mm_Vertical
Changed lines of the file:
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@@
       (effects (font (size 1.27 1.27)))
     )
-    (property "Footprint" "Connector_PinSocket_2.54mm:PinSocket_2x05_P2.54mm_Vertical" (at 123.19 81.28 0)
+    (property "Footprint" "Connector_PinHeader_2.54mm:PinHeader_2x05_P2.54mm_Vertical" (at 123.19 81.28 0)
       (effects (font (size 1.27 1.27)) hide)
     )
