File: boards/userioswitch/userioswitch.kicad_pcb (KiCad board)
At the start: 2 copper layers, 63 x 42 mm, 15 parts, among them IC1 SN3257QPWRQ1, IC2 SN3257QPWRQ1, J1 692112030100, J2 Conn_02x03_Odd_Even, J3 692122030100, J4 692122030100, J5 692122030100, J6 692122030100, J7 Conn_02x05_Odd_Even

Commit message: New
Parts:
- added R1: 4K7, Resistor_SMD:R_0805_2012Metric, F.Cu at (201.4, 90.8)
Routing:
- net VBUS: track 44.4 -> 46.6 mm
- net /SEL: track 29.0 -> 29.9 mm
Changed lines of the file:
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@@
     (property "Sheetname" "")
     (property "ki_description" "Wurth Elektronik WR-COM Series, Right Angle Through Hole, Version 3.0 Type A USB Connector, Receptacle")
-    (attr smd allow_missing_courtyard)
-    (fp_text reference "J4" (at 0 -2.032 90) (layer "F.SilkS")
-        (effects (font (size 1.27 1.27) (thickness 0.254)))
-    )
-    (fp_text value "692122030100" (at 0 2.669 90) (layer "F.SilkS") hide
-        (effects (font (size 1.27 1.27) (thickness 0.254)))
-    )
-    (fp_text user "${REFERENCE}" (at 0 2.669 90) (layer "F.Fab")
+    (attr smd)
+    (fp_text reference "J4" (at 0 2.669 -90) (layer "F.SilkS")
+        (effects (font (size 1.27 1.27) (thickness 0.254)))
+    )
+    (fp_text value "692122030100" (at 0 2.669 -90) (layer "F.SilkS") hide
+        (effects (font (size 1.27 1.27) (thickness 0.254)))
+    )
+    (fp_text user "${REFERENCE}" (at 0 2.669 -90) (layer "F.Fab")
         (effects (font (size 1.27 1.27) (thickness 0.254)))
     )
@@
     )
   )
+  (footprint "Resistor_SMD:R_0805_2012Metric" (layer "F.Cu")
+    (at 201.422 90.805)
+    (descr "Resistor SMD 0805 (2012 Metric), square (rectangular) end terminal, IPC_7351 nominal, (Body size source: IPC-SM-782 page 72, https://www.pcb-3d.com/wordpress/wp-content/uploads/ipc-sm-782a_amendment_1_and_2.pdf), generated with kicad-footprint-generator")
+    (tags "resistor")
+    (property "Sheetfile" "userioswitch.kicad_sch")
+    (property "Sheetname" "")
+    (property "ki_description" "Resistor")
+    (property "ki_keywords" "R res resistor")
+    (attr smd)
+    (fp_text reference "R1" (at 0 -1.65) (layer "F.SilkS")
+        (effects (font (size 1 1) (thickness 0.15)))
+    )
+    (fp_text value "4K7" (at 0 1.65) (layer "F.Fab")
+        (effects (font (size 1 1) (thickness 0.15)))
+    )
+    (fp_text user "${REFERENCE}" (at 0 0) (layer "F.Fab")
+        (effects (font (size 0.5 0.5) (thickness 0.08)))
+    )
+    (fp_line (start -0.227064 -0.735) (end 0.227064 -0.735)
+      (stroke (width 0.12) (type solid)) (layer "F.SilkS"))
+    (fp_line (start -0.227064 0.735) (end 0.227064 0.735)
+      (stroke (width 0.12) (type solid)) (layer "F.SilkS"))
+    (fp_line (start -1.68 -0.95) (end 1.68 -0.95)
+      (stroke (width 0.05) (type solid)) (layer "F.CrtYd"))
+    (fp_line (start -1.68 0.95) (end -1.68 -0.95)
+      (stroke (width 0.05) (type solid)) (layer "F.CrtYd"))
+    (fp_line (start 1.68 -0.95) (end 1.68 0.95)
+      (stroke (width 0.05) (type solid)) (layer "F.CrtYd"))
+    (fp_line (start 1.68 0.95) (end -1.68 0.95)
+      (stroke (width 0.05) (type solid)) (layer "F.CrtYd"))
+    (fp_line (start -1 -0.625) (end 1 -0.625)
+      (stroke (width 0.1) (type solid)) (layer "F.Fab"))
+    (fp_line (start -1 0.625) (end -1 -0.625)
+      (stroke (width 0.1) (type solid)) (layer "F.Fab"))
+    (fp_line (start 1 -0.625) (end 1 0.625)
+      (stroke (width 0.1) (type solid)) (layer "F.Fab"))
+    (fp_line (start 1 0.625) (end -1 0.625)
+      (stroke (width 0.1) (type solid)) (layer "F.Fab"))
+    (pad "1" smd roundrect (at -0.9125 0) (size 1.025 1.4) (layers "F.Cu" "F.Paste" "F.Mask") (roundrect_rratio 0.243902)
+      (net 1 "VBUS") (pintype "passive"))
+    (pad "2" smd roundrect (at 0.9125 0) (size 1.025 1.4) (layers "F.Cu" "F.Paste" "F.Mask") (roundrect_rratio 0.243902)
+      (net 3 "/SEL") (pintype "passive"))
+    (model "${KICAD6_3DMODEL_DIR}/Resistor_SMD.3dshapes/R_0805_2012Metric.wrl"
+      (offset (xyz 0 0 0))
+      (scale (xyz 1 1 1))
+      (rotate (xyz 0 0 0))
+    )
+  )
   (gr_rect (start 170.5 67) (end 233.5 109)
     (stroke (width 0.2) (type solid)) (fill none) (layer "Edge.Cuts"))
@@
   (segment (start 198.264 92.246) (end 198.562 91.948) (width 0.4) (layer "F.Cu") (net 1))
   (segment (start 212.786 90.358) (end 210.566 88.138) (width 0.4) (layer "F.Cu") (net 1))
+  (segment (start 199.131 90.805) (end 198.562 90.236) (width 0.254) (layer "F.Cu") (net 1))
   (segment (start 204.47 86.868) (end 201.93 86.868) (width 0.6) (layer "F.Cu") (net 1))
   (segment (start 210.566 88.138) (end 208.534 88.138) (width 0.4) (layer "F.Cu") (net 1))
   (segment (start 205.5339 100.076) (end 208.026 100.076) (width 0.6) (layer "F.Cu") (net 1))
+  (segment (start 200.5095 90.805) (end 199.131 90.805) (width 0.254) (layer "F.Cu") (net 1))
   (segment (start 207.7245 98.541) (end 208.026 98.2395) (width 0.4) (layer "F.Cu") (net 2))
   (segment (start 212.488 94.641) (end 212.463 94.616) (width 0.4) (layer "F.Cu") (net 2))
@@
   (segment (start 199.39 85.5031) (end 195.1669 85.5031) (width 0.25) (layer "F.Cu") (net 3))
   (segment (start 193.4506 93.991) (end 192.388 93.991) (width 0.25) (layer "F.Cu") (net 3))
-  (segment (start 206.3219 93.991) (end 206.612 93.991) (width 0.25) (layer "F.Cu") (net 3))
+  (segment (start 206.612 93.29655) (end 203.787225 90.471775) (width 0.25) (layer "F.Cu") (net 3))
   (segment (start 193.4506 87.2194) (end 193.4506 93.991) (width 0.25) (layer "F.Cu") (net 3))
   (segment (start 199.39 84.328) (end 199.39 85.5031) (width 0.25) (layer "F.Cu") (net 3))
   (segment (start 195.1669 85.5031) (end 193.4506 87.2194) (width 0.25) (layer "F.Cu") (net 3))
-  (segment (start 202.08845 89.75755) (end 206.3219 93.991) (width 0.25) (layer "F.Cu") (net 3))
-  (via (at 202.08845 89.75755) (size 0.8) (drill 0.4) (layers "F.Cu" "B.Cu") (net 3))
-  (segment (start 202.08845 89.75755) (end 200.5651 88.2342) (width 0.25) (layer "B.Cu") (net 3))
-  (segment (start 199.39 85.5031) (end 199.39 84.328) (width 0.25) (layer "B.Cu") (net 3))
-  (segment (start 200.5651 88.2342) (end 200.5651 85.8703) (width 0.25) (layer "B.Cu") (net 3))
-  (segment (start 200.1979 85.5031) (end 199.39 85.5031) (width 0.25) (layer "B.Cu") (net 3))
-  (segment (start 200.5651 85.8703) (end 200.1979 85.5031) (width 0.25) (layer "B.Cu") (net 3))
+  (segment (start 206.612 93.991) (end 206.612 93.29655) (width 0.25) (layer "F.Cu") (net 3))
+  (segment (start 203.787225 90.471775) (end 202.08845 88.773) (width 0.25) (layer "F.Cu") (net 3))
+  (segment (start 203.454 90.805) (end 203.787225 90.471775) (width 0.254) (layer "F.Cu") (net 3))
+  (segment (start 202.3345 90.805) (end 203.454 90.805) (width 0.254) (layer "F.Cu") (net 3))
+  (via (at 202.08845 88.773) (size 0.8) (drill 0.4) (layers "F.Cu" "B.Cu") (net 3))
+  (segment (start 200.5651 85.5031) (end 200.5651 87.24965) (width 0.25) (layer "B.Cu") (net 3))
+  (segment (start 199.39 84.328) (end 200.5651 85.5031) (width 0.25) (layer "B.Cu") (net 3))
+  (segment (start 200.5651 87.24965) (end 202.08845 88.773) (width 0.25) (layer "B.Cu") (net 3))
   (segment (start 172.8558 91.0318) (end 173.223 91.0318) (width 0.25) (layer "F.Cu") (net 4))
   (segment (start 172.0478 86.1343) (end 172.0478 90.2238) (width 0.25) (layer "F.Cu") (net 4))
