File: boards/userioswitchhdr/userioswitchhdr-prev.kicad_sch (KiCad schematic)
At the start: 13 parts, among them IC1 SN3257QPWRQ1, IC2 SN3257QPWRQ1, J1 Input, J2 Control_Power, J3 Output A, J4 Output B

Commit message: Pending updates
Parts:
- J1: value Input -> Header
- J2: value Control_Power -> Conn_02x03_Odd_Even
- J3: value Output A -> Header
- J4: value Output B -> Header
Other:
- moved on the sheet: H1, H2, H3, H4, J1, J3
