File: boards/userioswitchhdr/userioswitchhdr.kicad_pcb (KiCad board)
At the start: 2 copper layers, 49.6 x 38 mm, 13 parts, among them IC1 SN3257QPWRQ1, IC2 SN3257QPWRQ1, J1 Header, J2 Conn_02x03_Odd_Even, J3 Header, J4 Header

Commit message: Pending updates
Parts:
- J1: value Header -> Input
- J2: value Conn_02x03_Odd_Even -> Control_Power
- J3: value Header -> Output A
- J4: value Header -> Output B
- moved C1 11.5 mm to (205.1, 83.4), turned to 0 degrees
- moved IC1 11.0 mm to (201.5, 87.2)
- moved J2 8.00 mm to (199.4, 78.9)
- moved R1 7.77 mm to (195.3, 77.5)
- moved IC2 7.63 mm to (201.9, 96.6)
- moved C2 5.77 mm to (205.9, 92.7), turned to 0 degrees
Connections:
- IC1 pad 10: /S2B -> /S1B
- IC1 pad 11: /S2A -> /S1A
- IC1 pad 2: /S4A -> /S5A
- IC1 pad 3: /S4B -> /S5B
- IC1 pad 4: /D4 -> /D5
- IC1 pad 5: /S3A -> /S2A
- IC1 pad 6: /S3B -> /S2B
- IC1 pad 7: /D3 -> /D2
- IC1 pad 9: /D2 -> /D1
- IC2 pad 2: /S1A -> /S4A
- IC2 pad 3: /S1B -> /S4B
- IC2 pad 4: /D1 -> /D4
- IC2 pad 5: /S5A -> /S3A
- IC2 pad 6: /S5B -> /S3B
- IC2 pad 7: /D5 -> /D3
Routing:
- net VBUS: track 97.1 -> 0.00 mm, vias 2 -> 0
- net /VBUSB: track 41.1 -> 0.00 mm
- net /SEL: track 32.7 -> 0.00 mm, vias 2 -> 0
- net /VBUSA: track 23.6 -> 0.00 mm
- net /D2: track 8.73 -> 21.5 mm
- net /D5: track 10.9 -> 23.4 mm
- net /S5A: track 26.7 -> 17.5 mm
- net /S5B: track 18.4 -> 27.5 mm
- net /S6B: track 9.86 -> 17.7 mm, vias 0 -> 1
- net /S7B: track 9.62 -> 17.4 mm
- net /S6A: track 33.7 -> 41.0 mm
- net /S4A: track 9.62 -> 16.1 mm
- net /S3A: track 9.87 -> 16.3 mm
- net /S4B: track 33.8 -> 27.5 mm
- net /S3B: track 35.8 -> 30.7 mm, vias 1 -> 2
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