File: boards/userioswitchhdr/userioswitchhdr.kicad_sch (KiCad schematic)
At the start: 13 parts, among them IC1 SN3257QPWRQ1, IC2 SN3257QPWRQ1, J1 Header, J2 Conn_02x03_Odd_Even, J3 Header, J4 Header

Commit message: Pending updates
Parts:
- J1: value Header -> Input
- J2: value Conn_02x03_Odd_Even -> Control_Power
- J3: value Header -> Output A
- J4: value Header -> Output B
Connections:
- net D1: now also IC1.9 (D3); no longer IC2.4 (D1)
- net D2: now also IC1.7 (D2); no longer IC1.9 (D3)
- net D3: now also IC2.7 (D2); no longer IC1.7 (D2)
- net D4: now also IC2.4 (D1); no longer IC1.4 (D1)
- net D5: now also IC1.4 (D1); no longer IC2.7 (D2)
- net S1A: now also IC1.11 (S3A); no longer IC2.2 (S1A)
- net S1B: now also IC1.10 (S3B); no longer IC2.3 (S1B)
- net S2A: now also IC1.5 (S2A); no longer IC1.11 (S3A)
- net S2B: now also IC1.6 (S2B); no longer IC1.10 (S3B)
- net S3A: now also IC2.5 (S2A); no longer IC1.5 (S2A)
- net S3B: now also IC2.6 (S2B); no longer IC1.6 (S2B)
- net S4A: now also IC2.2 (S1A); no longer IC1.2 (S1A)
- net S4B: now also IC2.3 (S1B); no longer IC1.3 (S1B)
- net S5A: now also IC1.2 (S1A); no longer IC2.5 (S2A)
- net S5B: now also IC1.3 (S1B); no longer IC2.6 (S2B)
Other:
- moved on the sheet: H1, H2, H3, H4, J1, J3
