File: boards/picoio-lite/_autosave-picoio.kicad_pcb (KiCad board)
At the start: 2 copper layers, 108 x 77 mm, 33 parts, among them J1 Term, J10 VSYSIN, J12 ButtonLED, J13 OneWire, J14 Conn_01x04_Pin, J17 PI_USB, J18 12VBOOST, J19 ADCs, J2 Conn_01x02_Pin, J5 MiSTerLED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

Commit message: backups
Parts:
- added U4: TS3USB30EDGSR, Package_SO:VSSOP-10_3x3mm_P0.5mm, F.Cu at (124.3, 106.9)
- added U5: TS3USB30EDGSR, Package_SO:VSSOP-10_3x3mm_P0.5mm, F.Cu at (124.3, 111.5)
Connections:
- J17 pad 6: /USB_SWITCH_OC -> unconnected-(J17-Pin_6-Pad6)
- J17 pad 8: /USB_SWITCH_MON -> unconnected-(J17-Pin_8-Pad8)
- U3 pad 14: /USB_SWITCH_OC -> unconnected-(U3-O3-Pad14)
- U3 pad 3: /USB_SWITCH -> unconnected-(U3-I3-Pad3)
Routing:
- net /USB_SWITCH_OC: track 68.1 -> 0.00 mm
- net (no net): track 0.00 -> 68.1 mm
