File: boards/picoio-lite/picoio.kicad_sch (KiCad schematic)
At the start: 33 parts, among them J1 Term, J10 VSYSIN, J12 ButtonLED, J13 OneWire, J14 Conn_01x04_Pin, J17 PI_USB, J18 12VBOOST, J19 ADCs, J5 MiSTerLED, J6 MiSTerSwitch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

Commit message: backups
Parts:
- removed JP1: Jumper_2_Bridged, symbol Jumper:Jumper_2_Bridged
- added J2: Conn_01x02_Pin, Connector_PinHeader_2.54mm:PinHeader_1x02_P2.54mm_Vertical, symbol Connector:Conn_01x02_Pin
- added U4, U5: TS3USB30EDGSR, Package_SO:VSSOP-10_3x3mm_P0.5mm, symbol Interface_USB:TS3USB30EDGSR
- J8: footprint Connector_PinHeader_2.54mm:PinHeader_2x06_P2.54mm_Vertical -> Connector_PinHeader_2.54mm:PinHeader_2x04_P2.54mm_Vertical; symbol Connector_Generic:Conn_02x06_Odd_Even -> Connector_Generic:Conn_02x04_Odd_Even
Connections:
- net +3V3: now also U4.10 (VCC), U5.10 (VCC)
- net ADC2: now also J8.4 (Pin_4); no longer J8.8 (Pin_8)
- net DISPLAY_PWM: now also J8.6 (Pin_6); no longer J8.10 (Pin_10)
- net GND: now also U4.5 (GND), U5.5 (GND); no longer J8.11 (Pin_11), J8.9 (Pin_9)
- net USB_SWITCH: no longer U3.3 (I3)
- net USB_SWITCH_MON: no longer J17.8 (Pin_8)
- net VSYS: now also J2.2 (Pin_2)
- net VBUS: now reaches U1.40 (VBUS)
- net VBUS: now also J2.1 (Pin_1)
- net USB_SWITCH_OC: no longer names the net of J17.6 (Pin_6)
- net USB_SWITCH_OC: no longer U3.14 (O3)
- new net: U4.4 (D+), U5.2 (D1+)
- new net: U4.6 (D-), U5.8 (D1-)
- new net USBSW1: U4.1 (S)
- new net USBSW2: U5.1 (S)
- new net _USBSWOE: U4.9 (~{OE}), U5.9 (~{OE})
- no-connect marks 14 -> 13
